Commit message: Update robotic_arm.urdf

File: robotic_arm/urdf/robotic_arm.urdf (robot description, URDF)
Before this commit: robot robotic_arm, 9 links, 8 joints
Links:
- removed link world
- link base_link: mass 17.1466031047213 -> 17.147
- link link1: mass 3.09046329461166 -> 3.09046329461168
- link link3: mass 2.82619520385501 -> 2.82619520285645
- link link5: mass 0.190534240004917 -> 0.190534243496226
Joints:
- removed joint base_joint
- joint link2_revolute: axis 0 0 1 -> 0.0634251661005122 0 -0.997986597257259
- joint link3_revolute: axis 0 0 1 -> 0.0634160405786047 0.00107586811877688 -0.99798659725726
- joint link4_revolute: axis 0 0 1 -> -0.309036699346333 0 -0.95105011353615; limit lower=-3.142 upper=0 effort=0 velocity=0 -> lower=0 upper=-3.142 effort=0 velocity=0; origin xyz=0.0500000000000015 0.35 0 rpy=0 0 1.5707963267949 -> xyz=0.33669051723305 0.075138823425112 0.0916168806467064 rpy=0 -0.37764775167464 0.0169636090218595
- joint link5_revolute: axis 1 0 0 -> -0.0271031214688434 -0.00904142340899337 0.99959175340205; origin xyz=0.00200000000000555 0.800000000000001 0 rpy=3.14159265358979 0 0 -> xyz=0.0217512505054844 -0.225430946671694 -0.0806707591650744 rpy=1.50080931610212 0.0154073486983046 -2.92525450953042
- joint link6_1_prismatic: axis 0 0 1 -> -0.0010759 -0.063416 -0.99799; origin xyz=0 0 -0.01 rpy=0 0 0 -> xyz=0.91471 0.3654 0.76296 rpy=-1.5116 -1.3256 -2.8152
- joint link6_2_prismatic: axis 0 0 -1 -> -0.00107586811877956 0.0634160405786034 0.997986597257259; origin xyz=0 0.8 0.01 rpy=3.1416 0 0 -> xyz=0.203547969834237 0.0536399403068246 0.569409308513323 rpy=1.62995489797154 -1.32563166552103 -2.81517539067378

Commit message: Update robotic_arm.urdf

File: robotic_arm/urdf/robotic_arm.urdf (robot description, URDF)
Before this commit: robot robotic_arm, 8 links, 7 joints
Links:
- added link world
- link base_link: mass 17.147 -> 17.1466031047213
- link link1: mass 3.09046329461168 -> 3.09046329461166
- link link3: mass 2.82619520285645 -> 2.82619520385501
- link link5: mass 0.190534243496226 -> 0.190534240004917
Joints:
- added joint base_joint: type fixed, parent world, child base_link, origin xyz=0.0 0.0 0.0 rpy=0 0 0
- joint link2_revolute: axis 0.0634251661005122 0 -0.997986597257259 -> 0 0 1
- joint link3_revolute: axis 0.0634160405786047 0.00107586811877688 -0.99798659725726 -> 0 0 1
- joint link4_revolute: axis -0.309036699346333 0 -0.95105011353615 -> 0 0 1; limit lower=0 upper=-3.142 effort=0 velocity=0 -> lower=-3.142 upper=0 effort=0 velocity=0; origin xyz=0.33669051723305 0.075138823425112 0.0916168806467064 rpy=0 -0.37764775167464 0.0169636090218595 -> xyz=0.0500000000000015 0.35 0 rpy=0 0 1.5707963267949
- joint link5_revolute: axis -0.0271031214688434 -0.00904142340899337 0.99959175340205 -> 1 0 0; origin xyz=0.0217512505054844 -0.225430946671694 -0.0806707591650744 rpy=1.50080931610212 0.0154073486983046 -2.92525450953042 -> xyz=0.00200000000000555 0.800000000000001 0 rpy=3.14159265358979 0 0
- joint link6_1_prismatic: axis -0.0010759 -0.063416 -0.99799 -> 0 0 1; origin xyz=0.91471 0.3654 0.76296 rpy=-1.5116 -1.3256 -2.8152 -> xyz=0 0 -0.01 rpy=0 0 0
- joint link6_2_prismatic: axis -0.00107586811877956 0.0634160405786034 0.997986597257259 -> 0 0 -1; origin xyz=0.203547969834237 0.0536399403068246 0.569409308513323 rpy=1.62995489797154 -1.32563166552103 -2.81517539067378 -> xyz=0 0.8 0.01 rpy=3.1416 0 0
