Commit message: Update tractor.urdf

File: tractor/urdf/tractor.urdf (robot description, URDF)
Before this commit: robot tractor, 5 links, 4 joints
Joints:
- joint Front1: limit lower=-3.14 upper=3.14 effort=10 velocity=1 -> lower=0 upper=0 effort=0 velocity=0
- joint Front2: limit lower=-3.14 upper=3.14 effort=0 velocity=1 -> lower=0 upper=0 effort=0 velocity=0
- joint Rear1: limit lower=-3.14 upper=3.14 effort=10 velocity=1 -> lower=0 upper=0 effort=0 velocity=0
- joint Rear2: limit lower=-3.14 upper=3.14 effort=10 velocity=1 -> lower=0 upper=0 effort=0 velocity=0

Commit message: Update tractor.urdf

File: tractor/urdf/tractor.urdf (robot description, URDF)
Before this commit: robot tractor, 5 links, 4 joints
Links:
- link REAR_R: mass 3290 -> 0

Commit message: Update tractor.urdf

File: tractor/urdf/tractor.urdf (robot description, URDF)
Before this commit: robot tractor, 5 links, 4 joints
Joints:
- joint Front1: limit lower=0 upper=0 effort=0 velocity=0 -> (none)
- joint Front2: limit lower=0 upper=0 effort=0 velocity=0 -> (none)
- joint Rear1: limit lower=0 upper=0 effort=0 velocity=0 -> (none)
- joint Rear2: limit lower=0 upper=0 effort=0 velocity=0 -> (none)

Commit message: Update tractor.urdf

File: tractor/urdf/tractor.urdf (robot description, URDF)
Before this commit: robot tractor, 5 links, 4 joints
Joints:
- joint Front1: limit (none) -> lower=0 upper=0 effort=0 velocity=0
- joint Front2: limit (none) -> lower=0 upper=0 effort=0 velocity=0
- joint Rear1: limit (none) -> lower=0 upper=0 effort=0 velocity=0
- joint Rear2: limit (none) -> lower=0 upper=0 effort=0 velocity=0

Commit message: initial commit

File: tractor/urdf/tractor.urdf (robot description, URDF)
Before this commit: robot tractor, 6 links, 5 joints
Joints:
- joint implement: limit lower=-1 upper=1 effort=30 velocity=1 -> lower=0 upper=0 effort=0 velocity=1; type revolute -> fixed

Commit message: initial comm

File: tractor/urdf/tractor.urdf (robot description, URDF)
Before this commit: robot tractor, 6 links, 5 joints
Links:
- removed link IMPLEMENT
Joints:
- removed joint implement
